Commit message: Upload new worlds

File: urdf/robocop.xacro (robot description, xacro)
@@ -68,4 +68,23 @@
   </collision>
 </link>
+<link name="camera_auxiliar">
+  <inertial>
+      <inertia
+        ixx="0.166667" ixy="0" ixz="0"
+        iyx="0" iyy="0.166667" iyz="0"
+        izx="0" izy="0" izz="0.166667"
+        />
+    </inertial>
+    <visual name='visual'>
+      <geometry>
+        <box size="0.1 0.2 0.1" />
+      </geometry>
+    </visual>
+    <collision name='collision'>
+      <geometry>
+        <box size="0.1 0.2 0.1" />
+      </geometry>
+    </collision>
+</link>
 <link name="soporteElectronica_v7_1">
   <inertial>
@@ -513,3 +532,8 @@
   <axis xyz="1.0 -0.0 0.0"/>
 </joint>
+<joint name="robot_camera" type="fixed">
+  <origin xyz="0.0 -0.8 0.2" rpy="0 0 1.570795"/>
+  <parent link="depthCamera_v1_1"/>
+  <child link="camera_auxiliar"/>
+</joint>
 </robot>

Commit message: New launch values

File: urdf/robocop.xacro (robot description, xacro)
@@ -520,5 +520,5 @@
   <parent link="baseRuedas_v3_1"/>
   <child link="rueda_v2__4__1"/>
-  <axis xyz="1.0 -0.0 0.0"/>
+  <axis xyz="1.0 0.0 0.0"/>
 </joint>
 <joint name="ruedaDerecha4" type="continuous">
@@ -526,5 +526,5 @@
   <parent link="baseRuedas_v3_1"/>
   <child link="rueda_v2__3__1"/>
-  <axis xyz="1.0 -0.0 0.0"/>
+  <axis xyz="1.0 0.0 0.0"/>
 </joint>
 <joint name="ruedaDerecha3" type="continuous">
@@ -532,5 +532,5 @@
   <parent link="baseRuedas_v3_1"/>
   <child link="rueda_v2__2__1"/>
-  <axis xyz="1.0 -0.0 0.0"/>
+  <axis xyz="-1.0 -0.0 0.0"/>
 </joint>
 <joint name="ruedaDerecha2" type="continuous">
@@ -538,5 +538,5 @@
   <parent link="baseRuedas_v3_1"/>
   <child link="rueda_v2__1__1"/>
-  <axis xyz="1.0 -0.0 0.0"/>
+  <axis xyz="1.0 0.0 0.0"/>
 </joint>
 <joint name="ruedaDerecha1" type="continuous">
@@ -544,5 +544,5 @@
   <parent link="baseRuedas_v3_1"/>
   <child link="rueda_v2_1"/>
-  <axis xyz="1.0 -0.0 0.0"/>
+  <axis xyz="1.0 0.0 0.0"/>
 </joint>
 <joint name="R\EDgida94" type="fixed">

Commit message: upload data

File: urdf/robocop.xacro (robot description, xacro)
@@ -520,5 +520,5 @@
   <parent link="baseRuedas_v3_1"/>
   <child link="rueda_v2__4__1"/>
-  <axis xyz="1.0 0.0 0.0"/>
+  <axis xyz="-1.0 0.0 0.0"/>
 </joint>
 <joint name="ruedaDerecha4" type="continuous">
@@ -526,5 +526,5 @@
   <parent link="baseRuedas_v3_1"/>
   <child link="rueda_v2__3__1"/>
-  <axis xyz="1.0 0.0 0.0"/>
+  <axis xyz="-1.0 0.0 0.0"/>
 </joint>
 <joint name="ruedaDerecha3" type="continuous">
@@ -532,5 +532,5 @@
   <parent link="baseRuedas_v3_1"/>
   <child link="rueda_v2__2__1"/>
-  <axis xyz="-1.0 -0.0 0.0"/>
+  <axis xyz="-1.0 0.0 0.0"/>
 </joint>
 <joint name="ruedaDerecha2" type="continuous">
@@ -538,5 +538,5 @@
   <parent link="baseRuedas_v3_1"/>
   <child link="rueda_v2__1__1"/>
-  <axis xyz="1.0 0.0 0.0"/>
+  <axis xyz="-1.0 0.0 0.0"/>
 </joint>
 <joint name="ruedaDerecha1" type="continuous">
@@ -544,7 +544,7 @@
   <parent link="baseRuedas_v3_1"/>
   <child link="rueda_v2_1"/>
-  <axis xyz="1.0 0.0 0.0"/>
-</joint>
-<joint name="R\EDgida94" type="fixed">
+  <axis xyz="-1.0 0.0 0.0"/>
+</joint>
+<joint name="Rigida94" type="fixed">
   <origin xyz="0.0757 0.117 0.068" rpy="0 0 0"/>
   <parent link="soporteElectronica_v7_1"/>

Commit message: change robocop model

File: urdf/robocop.xacro (robot description, xacro)
@@ -490,5 +490,5 @@
   <parent link="baseRuedas_v3__1__1"/>
   <child link="rueda_v2__9__1"/>
-  <axis xyz="-1.0 0.0 0.0"/>
+  <axis xyz="1.0 0.0 0.0"/>
 </joint>
 <joint name="ruedaIzquierda2" type="continuous">
@@ -496,5 +496,5 @@
   <parent link="baseRuedas_v3__1__1"/>
   <child link="rueda_v2__8__1"/>
-  <axis xyz="-1.0 0.0 0.0"/>
+  <axis xyz="1.0 0.0 0.0"/>
 </joint>
 <joint name="ruedaIzquierda3" type="continuous">
@@ -502,5 +502,5 @@
   <parent link="baseRuedas_v3__1__1"/>
   <child link="rueda_v2__7__1"/>
-  <axis xyz="-1.0 0.0 0.0"/>
+  <axis xyz="1.0 0.0 0.0"/>
 </joint>
 <joint name="ruedaIzquierda4" type="continuous">
@@ -508,5 +508,5 @@
   <parent link="baseRuedas_v3__1__1"/>
   <child link="rueda_v2__6__1"/>
-  <axis xyz="-1.0 0.0 0.0"/>
+  <axis xyz="1.0 0.0 0.0"/>
 </joint>
 <joint name="ruedaIzquierda5" type="continuous">
@@ -514,5 +514,5 @@
   <parent link="baseRuedas_v3__1__1"/>
   <child link="rueda_v2__5__1"/>
-  <axis xyz="-1.0 0.0 0.0"/>
+  <axis xyz="1.0 0.0 0.0"/>
 </joint>
 <joint name="ruedaDerecha5" type="continuous">
@@ -520,5 +520,5 @@
   <parent link="baseRuedas_v3_1"/>
   <child link="rueda_v2__4__1"/>
-  <axis xyz="-1.0 0.0 0.0"/>
+  <axis xyz="1.0 0.0 0.0"/>
 </joint>
 <joint name="ruedaDerecha4" type="continuous">
@@ -526,5 +526,5 @@
   <parent link="baseRuedas_v3_1"/>
   <child link="rueda_v2__3__1"/>
-  <axis xyz="-1.0 0.0 0.0"/>
+  <axis xyz="1.0 0.0 0.0"/>
 </joint>
 <joint name="ruedaDerecha3" type="continuous">
@@ -532,5 +532,5 @@
   <parent link="baseRuedas_v3_1"/>
   <child link="rueda_v2__2__1"/>
-  <axis xyz="-1.0 0.0 0.0"/>
+  <axis xyz="1.0 0.0 0.0"/>
 </joint>
 <joint name="ruedaDerecha2" type="continuous">
@@ -538,5 +538,5 @@
   <parent link="baseRuedas_v3_1"/>
   <child link="rueda_v2__1__1"/>
-  <axis xyz="-1.0 0.0 0.0"/>
+  <axis xyz="1.0 0.0 0.0"/>
 </joint>
 <joint name="ruedaDerecha1" type="continuous">
@@ -544,5 +544,5 @@
   <parent link="baseRuedas_v3_1"/>
   <child link="rueda_v2_1"/>
-  <axis xyz="-1.0 0.0 0.0"/>
+  <axis xyz="1.0 0.0 0.0"/>
 </joint>
 <joint name="Rigida94" type="fixed">
