Commit message: Upload new model

File: urdf/materials.xacro (robot description, xacro)
@@ -16,3 +16,9 @@
   <color rgba="0.9098039215686274 0.44313725490196076 0.03137254901960784 1.0"/>
 </material>
+<material name="plstico_brillante_negro">
+  <color rgba="0.09803921568627451 0.09803921568627451 0.09803921568627451 1.0"/>
+</material>
+<material name="aluminio_anodizado_rugoso_gris">
+  <color rgba="0.5372549019607843 0.5372549019607843 0.5372549019607843 1.0"/>
+</material>
 </robot>

File: urdf/robocop.xacro (robot description, xacro)
@@ -8,7 +8,7 @@
 <link name="base_link">
   <inertial>
-    <origin xyz="0.0018651922128957463 -0.0001339941880531507 0.08792532537696136" rpy="0 0 0"/>
+    <origin xyz="-0.0013001515328987126 -0.0017028571084608795 0.08695702362938688" rpy="0 0 0"/>
     <mass value="0.518865961499241"/>
-    <inertia ixx="0.002526" iyy="0.001389" izz="0.003913" ixy="-0.0" iyz="0.0" ixz="-0.0"/>
+    <inertia ixx="0.002526" iyy="0.001389" izz="0.003913" ixy="-0.0" iyz="0.0" ixz="0.0"/>
   </inertial>
   <visual>
@@ -28,10 +28,10 @@
 <link name="soporteCamara_v2_1">
   <inertial>
-    <origin xyz="0.031000192212050377 0.03309723523847037 0.0028231628652582857" rpy="0 0 0"/>
+    <origin xyz="0.030999848466254507 0.03309637231806288 0.0028238611176833878" rpy="0 0 0"/>
     <mass value="0.3066668323515448"/>
     <inertia ixx="0.000213" iyy="0.000189" izz="0.0004" ixy="0.0" iyz="-4e-06" ixz="0.0"/>
   </inertial>
   <visual>
-    <origin xyz="0.029135 -0.089863 -0.090415" rpy="0 0 0"/>
+    <origin xyz="0.0323 -0.088295 -0.089446" rpy="0 0 0"/>
     <geometry>
       <mesh filename="package://robocop_description/meshes/soporteCamara_v2_1.stl" scale="0.001 0.001 0.001"/>
@@ -40,5 +40,5 @@
   </visual>
   <collision>
-    <origin xyz="0.029135 -0.089863 -0.090415" rpy="0 0 0"/>
+    <origin xyz="0.0323 -0.088295 -0.089446" rpy="0 0 0"/>
     <geometry>
       <mesh filename="package://robocop_description/meshes/soporteCamara_v2_1.stl" scale="0.001 0.001 0.001"/>
@@ -48,10 +48,10 @@
 <link name="depthCamera_v1_1">
   <inertial>
-    <origin xyz="1.3321708433653053e-05 -0.013660163121100521 0.013864662196538036" rpy="0 0 0"/>
+    <origin xyz="1.2977962637454295e-05 -0.013660026041507928 0.013865360448962805" rpy="0 0 0"/>
     <mass value="1.4328260381707594"/>
     <inertia ixx="0.000283" iyy="0.003111" izz="0.00318" ixy="-0.0" iyz="-5e-06" ixz="-0.0"/>
   </inertial>
   <visual>
-    <origin xyz="-0.001865 -0.165189 -0.098881" rpy="0 0 0"/>
+    <origin xyz="0.0013 -0.16362 -0.097912" rpy="0 0 0"/>
     <geometry>
       <mesh filename="package://robocop_description/meshes/depthCamera_v1_1.stl" scale="0.001 0.001 0.001"/>
@@ -60,5 +60,5 @@
   </visual>
   <collision>
-    <origin xyz="-0.001865 -0.165189 -0.098881" rpy="0 0 0"/>
+    <origin xyz="0.0013 -0.16362 -0.097912" rpy="0 0 0"/>
     <geometry>
       <mesh filename="package://robocop_description/meshes/depthCamera_v1_1.stl" scale="0.001 0.001 0.001"/>
@@ -68,10 +68,10 @@
 <link name="soporteElectronica_v7_1">
   <inertial>
-    <origin xyz="0.07505366903855869 0.05500321236476466 0.04613542479954183" rpy="0 0 0"/>
+    <origin xyz="0.07505332529276447 0.055002349444357466 0.04613612305196724" rpy="0 0 0"/>
     <mass value="1.7280541618979528"/>
     <inertia ixx="0.002669" iyy="0.008802" izz="0.009606" ixy="0.0" iyz="-0.0" ixz="2.2e-05"/>
   </inertial>
   <visual>
-    <origin xyz="0.073835 0.055137 -0.090415" rpy="0 0 0"/>
+    <origin xyz="0.077 0.056705 -0.089446" rpy="0 0 0"/>
     <geometry>
       <mesh filename="package://robocop_description/meshes/soporteElectronica_v7_1.stl" scale="0.001 0.001 0.001"/>
@@ -80,5 +80,5 @@
   </visual>
   <collision>
-    <origin xyz="0.073835 0.055137 -0.090415" rpy="0 0 0"/>
+    <origin xyz="0.077 0.056705 -0.089446" rpy="0 0 0"/>
     <geometry>
       <mesh filename="package://robocop_description/meshes/soporteElectronica_v7_1.stl" scale="0.001 0.001 0.001"/>
@@ -86,32 +86,12 @@
   </collision>
 </link>
-<link name="LIDAR_v1_1">
-  <inertial>
-    <origin xyz="1.922129045869598e-07 -0.04935393654029111 0.033571184302419205" rpy="0 0 0"/>
-    <mass value="0.6325892936987738"/>
-    <inertia ixx="0.000422" iyy="0.000181" izz="0.000485" ixy="-0.0" iyz="-6.5e-05" ixz="0.0"/>
-  </inertial>
-  <visual>
-    <origin xyz="-0.000865 -0.041663 -0.155415" rpy="0 0 0"/>
-    <geometry>
-      <mesh filename="package://robocop_description/meshes/LIDAR_v1_1.stl" scale="0.001 0.001 0.001"/>
-    </geometry>
-    <material name="acero_satinado"/>
-  </visual>
-  <collision>
-    <origin xyz="-0.000865 -0.041663 -0.155415" rpy="0 0 0"/>
-    <geometry>
-      <mesh filename="package://robocop_description/meshes/LIDAR_v1_1.stl" scale="0.001 0.001 0.001"/>
-    </geometry>
-  </collision>
-</link>
 <link name="basePrincipal_v4_1">
   <inertial>
-    <origin xyz="0.06750019221290116 -0.08999961693977199 -0.0010003687853090693" rpy="0 0 0"/>
+    <origin xyz="0.0674998484671067 -0.09000047986017973 -0.0009996705328835231" rpy="0 0 0"/>
     <mass value="0.44398234905881495"/>
-    <inertia ixx="0.001466" iyy="0.000868" izz="0.002334" ixy="-0.0" iyz="-0.0" ixz="-0.0"/>
-  </inertial>
-  <visual>
-    <origin xyz="0.065635 -0.089863 -0.085415" rpy="0 0 0"/>
+    <inertia ixx="0.001466" iyy="0.000868" izz="0.002334" ixy="-0.0" iyz="0.0" ixz="0.0"/>
+  </inertial>
+  <visual>
+    <origin xyz="0.0688 -0.088295 -0.084446" rpy="0 0 0"/>
     <geometry>
       <mesh filename="package://robocop_description/meshes/basePrincipal_v4_1.stl" scale="0.001 0.001 0.001"/>
@@ -120,5 +100,5 @@
   </visual>
   <collision>
-    <origin xyz="0.065635 -0.089863 -0.085415" rpy="0 0 0"/>
+    <origin xyz="0.0688 -0.088295 -0.084446" rpy="0 0 0"/>
     <geometry>
       <mesh filename="package://robocop_description/meshes/basePrincipal_v4_1.stl" scale="0.001 0.001 0.001"/>
@@ -128,10 +108,10 @@
 <link name="baseRuedas_v3__1__1">
   <inertial>
-    <origin xyz="-0.002915597767569167 -0.00016114326254506946 -0.03517882493390456" rpy="0 0 0"/>
+    <origin xyz="-0.0029159415133633293 -0.0001620061829542209 -0.035178126681478745" rpy="0 0 0"/>
     <mass value="0.25465013251117524"/>
     <inertia ixx="0.001194" iyy="0.000128" izz="0.001072" ixy="-0.0" iyz="4e-06" ixz="-9e-06"/>
   </inertial>
   <visual>
-    <origin xyz="0.073135 0.000137 -0.083415" rpy="0 0 0"/>
+    <origin xyz="0.0763 0.001705 -0.082446" rpy="0 0 0"/>
     <geometry>
       <mesh filename="package://robocop_description/meshes/baseRuedas_v3__1__1.stl" scale="0.001 0.001 0.001"/>
@@ -140,5 +120,5 @@
   </visual>
   <collision>
-    <origin xyz="0.073135 0.000137 -0.083415" rpy="0 0 0"/>
+    <origin xyz="0.0763 0.001705 -0.082446" rpy="0 0 0"/>
     <geometry>
       <mesh filename="package://robocop_description/meshes/baseRuedas_v3__1__1.stl" scale="0.001 0.001 0.001"/>
@@ -148,10 +128,10 @@
 <link name="baseRuedas_v3_1">
   <inertial>
-    <origin xyz="0.003915982193377993 0.0001619093830012282 -0.03517882493390446" rpy="0 0 0"/>
+    <origin xyz="0.003915638447583289 0.0001610464625932985 -0.035178126681478884" rpy="0 0 0"/>
     <mass value="0.25465013251117524"/>
     <inertia ixx="0.001194" iyy="0.000128" izz="0.001072" ixy="-0.0" iyz="-4e-06" ixz="9e-06"/>
   </inertial>
   <visual>
-    <origin xyz="-0.076865 0.000137 -0.083415" rpy="0 0 0"/>
+    <origin xyz="-0.0737 0.001705 -0.082446" rpy="0 0 0"/>
     <geometry>
       <mesh filename="package://robocop_description/meshes/baseRuedas_v3_1.stl" scale="0.001 0.001 0.001"/>
@@ -160,5 +140,5 @@
   </visual>
   <collision>
-    <origin xyz="-0.076865 0.000137 -0.083415" rpy="0 0 0"/>
+    <origin xyz="-0.0737 0.001705 -0.082446" rpy="0 0 0"/>
     <geometry>
       <mesh filename="package://robocop_description/meshes/baseRuedas_v3_1.stl" scale="0.001 0.001 0.001"/>
@@ -168,10 +148,10 @@
 <link name="soportePantalla_v11_1">
   <inertial>
-    <origin xyz="0.031024040064657452 -0.05481958862267361 0.0416925237926655" rpy="0 0 0"/>
+    <origin xyz="0.0310236963188651 -0.054820451543081225 0.04169322204509168" rpy="0 0 0"/>
     <mass value="1.4723320792485302"/>
     <inertia ixx="0.003175" iyy="0.003919" izz="0.002641" ixy="-1e-06" iyz="0.000192" ixz="1e-06"/>
   </inertial>
   <visual>
-    <origin xyz="0.029135 0.090137 -0.090415" rpy="0 0 0"/>
+    <origin xyz="0.0323 0.091705 -0.089446" rpy="0 0 0"/>
     <geometry>
       <mesh filename="package://robocop_description/meshes/soportePantalla_v11_1.stl" scale="0.001 0.001 0.001"/>
@@ -180,5 +160,5 @@
   </visual>
   <collision>
-    <origin xyz="0.029135 0.090137 -0.090415" rpy="0 0 0"/>
+    <origin xyz="0.0323 0.091705 -0.089446" rpy="0 0 0"/>
     <geometry>
       <mesh filename="package://robocop_description/meshes/soportePantalla_v11_1.stl" scale="0.001 0.001 0.001"/>
@@ -188,10 +168,10 @@
 <link name="pantallaTouch_v1_1">
   <inertial>
-    <origin xyz="0.05700911899382228 -0.021369246136639014 -0.03552692822423634" rpy="0 0 0"/>
+    <origin xyz="0.057008775248030316 -0.021370109057047254 -0.03552722997181007" rpy="0 0 0"/>
     <mass value="0.4448049684188369"/>
     <inertia ixx="0.000218" iyy="0.000719" izz="0.00059" ixy="0.0" iyz="-8.6e-05" ixz="0.0"/>
   </inertial>
   <visual>
-    <origin xyz="0.055135 0.136312 -0.224749" rpy="0 0 0"/>
+    <origin xyz="0.0583 0.13788 -0.223781" rpy="0 0 0"/>
     <geometry>
       <mesh filename="package://robocop_description/meshes/pantallaTouch_v1_1.stl" scale="0.001 0.001 0.001"/>
@@ -200,5 +180,5 @@
   </visual>
   <collision>
-    <origin xyz="0.055135 0.136312 -0.224749" rpy="0 0 0"/>
+    <origin xyz="0.0583 0.13788 -0.223781" rpy="0 0 0"/>
     <geometry>
       <mesh filename="package://robocop_description/meshes/pantallaTouch_v1_1.stl" scale="0.001 0.001 0.001"/>
@@ -208,10 +188,10 @@
 <link name="rueda_v2__9__1">
   <inertial>
-    <origin xyz="-0.024841290924186132 -1.7478473850196519e-07 3.995464235781454e-07" rpy="0 0 0"/>
+    <origin xyz="-0.024841634669981155 -3.770514719891871e-08 9.779884919958182e-08" rpy="0 0 0"/>
     <mass value="0.03535675163245145"/>
     <inertia ixx="5e-06" iyy="6e-06" izz="6e-06" ixy="-0.0" iyz="-0.0" ixz="-0.0"/>
   </inertial>
   <visual>
-    <origin xyz="0.076135 -0.106236 -0.034881" rpy="0 0 0"/>
+    <origin xyz="0.0793 -0.104667 -0.033913" rpy="0 0 0"/>
     <geometry>
       <mesh filename="package://robocop_description/meshes/rueda_v2__9__1.stl" scale="0.001 0.001 0.001"/>
@@ -220,5 +200,5 @@
   </visual>
   <collision>
-    <origin xyz="0.076135 -0.106236 -0.034881" rpy="0 0 0"/>
+    <origin xyz="0.0793 -0.104667 -0.033913" rpy="0 0 0"/>
     <geometry>
       <mesh filename="package://robocop_description/meshes/rueda_v2__9__1.stl" scale="0.001 0.001 0.001"/>
@@ -228,10 +208,10 @@
 <link name="rueda_v2__8__1">
   <inertial>
-    <origin xyz="-0.02484129092418627 3.830602414781059e-07 -3.6878536288295627e-07" rpy="0 0 0"/>
+    <origin xyz="-0.02484163466998078 -4.79860167851287e-07 3.294670629823415e-07" rpy="0 0 0"/>
     <mass value="0.03535675163245145"/>
     <inertia ixx="5e-06" iyy="6e-06" izz="6e-06" ixy="-0.0" iyz="-0.0" ixz="-0.0"/>
   </inertial>
   <visual>
-    <origin xyz="0.076135 -0.049863 -0.020415" rpy="0 0 0"/>
+    <origin xyz="0.0793 -0.048295 -0.019446" rpy="0 0 0"/>
     <geometry>
       <mesh filename="package://robocop_description/meshes/rueda_v2__8__1.stl" scale="0.001 0.001 0.001"/>
@@ -240,5 +220,5 @@
   </visual>
   <collision>
-    <origin xyz="0.076135 -0.049863 -0.020415" rpy="0 0 0"/>
+    <origin xyz="0.0793 -0.048295 -0.019446" rpy="0 0 0"/>
     <geometry>
       <mesh filename="package://robocop_description/meshes/rueda_v2__8__1.stl" scale="0.001 0.001 0.001"/>
@@ -248,10 +228,10 @@
 <link name="rueda_v2__7__1">
   <inertial>
-    <origin xyz="-0.024841290924185494 3.830602412746554e-07 -3.6878536301479525e-07" rpy="0 0 0"/>
+    <origin xyz="-0.02484163466997956 -4.798601685970013e-07 3.294670627949914e-07" rpy="0 0 0"/>
     <mass value="0.03535675163245145"/>
     <inertia ixx="5e-06" iyy="6e-06" izz="6e-06" ixy="-0.0" iyz="-0.0" ixz="-0.0"/>
   </inertial>
   <visual>
-    <origin xyz="0.076135 0.000137 -0.020415" rpy="0 0 0"/>
+    <origin xyz="0.0793 0.001705 -0.019446" rpy="0 0 0"/>
     <geometry>
       <mesh filename="package://robocop_description/meshes/rueda_v2__7__1.stl" scale="0.001 0.001 0.001"/>
@@ -260,5 +240,5 @@
   </visual>
   <collision>
-    <origin xyz="0.076135 0.000137 -0.020415" rpy="0 0 0"/>
+    <origin xyz="0.0793 0.001705 -0.019446" rpy="0 0 0"/>
     <geometry>
       <mesh filename="package://robocop_description/meshes/rueda_v2__7__1.stl" scale="0.001 0.001 0.001"/>
@@ -268,10 +248,10 @@
 <link name="rueda_v2__6__1">
   <inertial>
-    <origin xyz="-0.02484129092418562 3.8306024076339984e-07 -3.6878536291765074e-07" rpy="0 0 0"/>
+    <origin xyz="-0.02484163466997924 -4.798601688643656e-07 3.29467063017036e-07" rpy="0 0 0"/>
     <mass value="0.03535675163245145"/>
     <inertia ixx="5e-06" iyy="6e-06" izz="6e-06" ixy="-0.0" iyz="-0.0" ixz="-0.0"/>
   </inertial>
   <visual>
-    <origin xyz="0.076135 0.050137 -0.020415" rpy="0 0 0"/>
+    <origin xyz="0.0793 0.051705 -0.019446" rpy="0 0 0"/>
     <geometry>
       <mesh filename="package://robocop_description/meshes/rueda_v2__6__1.stl" scale="0.001 0.001 0.001"/>
@@ -280,5 +260,5 @@
   </visual>
   <collision>
-    <origin xyz="0.076135 0.050137 -0.020415" rpy="0 0 0"/>
+    <origin xyz="0.0793 0.051705 -0.019446" rpy="0 0 0"/>
     <geometry>
       <mesh filename="package://robocop_description/meshes/rueda_v2__6__1.stl" scale="0.001 0.001 0.001"/>
@@ -288,10 +268,10 @@
 <link name="rueda_v2__5__1">
   <inertial>
-    <origin xyz="-0.024841290924184245 3.830602405829886e-07 -3.687853628794868e-07" rpy="0 0 0"/>
+    <origin xyz="-0.024841634669977394 -4.798601686839543e-07 3.2946706300662765e-07" rpy="0 0 0"/>
     <mass value="0.03535675163245145"/>
     <inertia ixx="5e-06" iyy="6e-06" izz="6e-06" ixy="-0.0" iyz="-0.0" ixz="-0.0"/>
   </inertial>
   <visual>
-    <origin xyz="0.076135 0.100137 -0.033415" rpy="0 0 0"/>
+    <origin xyz="0.0793 0.101705 -0.032446" rpy="0 0 0"/>
     <geometry>
       <mesh filename="package://robocop_description/meshes/rueda_v2__5__1.stl" scale="0.001 0.001 0.001"/>
@@ -300,5 +280,5 @@
   </visual>
   <collision>
-    <origin xyz="0.076135 0.100137 -0.033415" rpy="0 0 0"/>
+    <origin xyz="0.0793 0.101705 -0.032446" rpy="0 0 0"/>
     <geometry>
       <mesh filename="package://robocop_description/meshes/rueda_v2__5__1.stl" scale="0.001 0.001 0.001"/>
@@ -308,10 +288,10 @@
 <link name="rueda_v2__4__1">
   <inertial>
-    <origin xyz="0.024841675349993597 -5.909477911181238e-08 3.9954653360124714e-07" rpy="0 0 0"/>
+    <origin xyz="0.024841331604199823 7.798481313492367e-08 9.779895947942263e-08" rpy="0 0 0"/>
     <mass value="0.03535675163245145"/>
     <inertia ixx="5e-06" iyy="6e-06" izz="6e-06" ixy="0.0" iyz="0.0" ixz="-0.0"/>
   </inertial>
   <visual>
-    <origin xyz="-0.080865 0.106509 -0.034881" rpy="0 0 0"/>
+    <origin xyz="-0.0777 0.108078 -0.033913" rpy="0 0 0"/>
     <geometry>
       <mesh filename="package://robocop_description/meshes/rueda_v2__4__1.stl" scale="0.001 0.001 0.001"/>
@@ -320,5 +300,5 @@
   </visual>
   <collision>
-    <origin xyz="-0.080865 0.106509 -0.034881" rpy="0 0 0"/>
+    <origin xyz="-0.0777 0.108078 -0.033913" rpy="0 0 0"/>
     <geometry>
       <mesh filename="package://robocop_description/meshes/rueda_v2__4__1.stl" scale="0.001 0.001 0.001"/>
@@ -328,10 +308,10 @@
 <link name="rueda_v2__3__1">
   <inertial>
-    <origin xyz="0.024841675349993916 3.8306024099238334e-07 -3.6878525307496024e-07" rpy="0 0 0"/>
+    <origin xyz="0.024841331604199518 -4.798601671712754e-07 3.2946717271054027e-07" rpy="0 0 0"/>
     <mass value="0.03535675163245145"/>
     <inertia ixx="5e-06" iyy="6e-06" izz="6e-06" ixy="0.0" iyz="0.0" ixz="-0.0"/>
   </inertial>
   <visual>
-    <origin xyz="-0.080865 0.050137 -0.020415" rpy="0 0 0"/>
+    <origin xyz="-0.0777 0.051705 -0.019446" rpy="0 0 0"/>
     <geometry>
       <mesh filename="package://robocop_description/meshes/rueda_v2__3__1.stl" scale="0.001 0.001 0.001"/>
@@ -340,5 +320,5 @@
   </visual>
   <collision>
-    <origin xyz="-0.080865 0.050137 -0.020415" rpy="0 0 0"/>
+    <origin xyz="-0.0777 0.051705 -0.019446" rpy="0 0 0"/>
     <geometry>
       <mesh filename="package://robocop_description/meshes/rueda_v2__3__1.stl" scale="0.001 0.001 0.001"/>
@@ -348,10 +328,10 @@
 <link name="rueda_v2__2__1">
   <inertial>
-    <origin xyz="0.02484167534999379 3.8306024162783423e-07 -3.687852531616964e-07" rpy="0 0 0"/>
+    <origin xyz="0.024841331604198866 -4.798601663451134e-07 3.2946717246420953e-07" rpy="0 0 0"/>
     <mass value="0.03535675163245145"/>
     <inertia ixx="5e-06" iyy="6e-06" izz="6e-06" ixy="0.0" iyz="0.0" ixz="-0.0"/>
   </inertial>
   <visual>
-    <origin xyz="-0.080865 0.000137 -0.020415" rpy="0 0 0"/>
+    <origin xyz="-0.0777 0.001705 -0.019446" rpy="0 0 0"/>
     <geometry>
       <mesh filename="package://robocop_description/meshes/rueda_v2__2__1.stl" scale="0.001 0.001 0.001"/>
@@ -360,5 +340,5 @@
   </visual>
   <collision>
-    <origin xyz="-0.080865 0.000137 -0.020415" rpy="0 0 0"/>
+    <origin xyz="-0.0777 0.001705 -0.019446" rpy="0 0 0"/>
     <geometry>
       <mesh filename="package://robocop_description/meshes/rueda_v2__2__1.stl" scale="0.001 0.001 0.001"/>
@@ -368,10 +348,10 @@
 <link name="rueda_v2__1__1">
   <inertial>
-    <origin xyz="0.02484167534999379 3.830602419707674e-07 -3.6878525317210475e-07" rpy="0 0 0"/>
+    <origin xyz="0.02484133160419831 -4.798601659430912e-07 3.2946717221440935e-07" rpy="0 0 0"/>
     <mass value="0.03535675163245145"/>
     <inertia ixx="5e-06" iyy="6e-06" izz="6e-06" ixy="0.0" iyz="0.0" ixz="-0.0"/>
   </inertial>
   <visual>
-    <origin xyz="-0.080865 -0.049863 -0.020415" rpy="0 0 0"/>
+    <origin xyz="-0.0777 -0.048295 -0.019446" rpy="0 0 0"/>
     <geometry>
       <mesh filename="package://robocop_description/meshes/rueda_v2__1__1.stl" scale="0.001 0.001 0.001"/>
@@ -380,5 +360,5 @@
   </visual>
   <collision>
-    <origin xyz="-0.080865 -0.049863 -0.020415" rpy="0 0 0"/>
+    <origin xyz="-0.0777 -0.048295 -0.019446" rpy="0 0 0"/>
     <geometry>
       <mesh filename="package://robocop_description/meshes/rueda_v2__1__1.stl" scale="0.001 0.001 0.001"/>
@@ -388,10 +368,10 @@
 <link name="rueda_v2_1">
   <inertial>
-    <origin xyz="0.024841675349992876 3.8306024210954526e-07 -3.687852527245461e-07" rpy="0 0 0"/>
+    <origin xyz="0.024841331604196965 -4.798601649924628e-07 3.294671725578846e-07" rpy="0 0 0"/>
     <mass value="0.03535675163245145"/>
     <inertia ixx="5e-06" iyy="6e-06" izz="6e-06" ixy="0.0" iyz="0.0" ixz="-0.0"/>
   </inertial>
   <visual>
-    <origin xyz="-0.080865 -0.099863 -0.033415" rpy="0 0 0"/>
+    <origin xyz="-0.0777 -0.098295 -0.032446" rpy="0 0 0"/>
     <geometry>
       <mesh filename="package://robocop_description/meshes/rueda_v2_1.stl" scale="0.001 0.001 0.001"/>
@@ -400,5 +380,5 @@
   </visual>
   <collision>
-    <origin xyz="-0.080865 -0.099863 -0.033415" rpy="0 0 0"/>
+    <origin xyz="-0.0777 -0.098295 -0.032446" rpy="0 0 0"/>
     <geometry>
       <mesh filename="package://robocop_description/meshes/rueda_v2_1.stl" scale="0.001 0.001 0.001"/>
@@ -406,26 +386,81 @@
   </collision>
 </link>
+<link name="Lidar_LD19_v1_1">
+  <inertial>
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