Commit message: Navigation stack update

File: urdf/materials.xacro (robot description, xacro)
@@ -19,6 +19,3 @@
   <color rgba="0.09803921568627451 0.09803921568627451 0.09803921568627451 1.0"/>
 </material>
-<material name="aluminio_anodizado_rugoso_gris">
-  <color rgba="0.5372549019607843 0.5372549019607843 0.5372549019607843 1.0"/>
-</material>
 </robot>

File: urdf/robocop.xacro (robot description, xacro)
@@ -8,7 +8,7 @@
 <link name="base_link">
   <inertial>
-    <origin xyz="-0.0013001515328987126 -0.0017028571084608795 0.08695702362938688" rpy="0 0 0"/>
-    <mass value="0.518865961499241"/>
-    <inertia ixx="0.002526" iyy="0.001389" izz="0.003913" ixy="-0.0" iyz="0.0" ixz="0.0"/>
+    <origin xyz="-0.00015252878117210557 0.0011495201398277505 0.08695702362938718" rpy="0 0 0"/>
+    <mass value="0.5188659614992409"/>
+    <inertia ixx="0.001389" iyy="0.002526" izz="0.003913" ixy="0.0" iyz="0.0" ixz="0.0"/>
   </inertial>
   <visual>
@@ -28,10 +28,10 @@
 <link name="soporteCamara_v2_1">
   <inertial>
-    <origin xyz="0.030999848466254507 0.03309637231806288 0.0028238611176833878" rpy="0 0 0"/>
-    <mass value="0.3066668323515448"/>
-    <inertia ixx="0.000213" iyy="0.000189" izz="0.0004" ixy="0.0" iyz="-4e-06" ixz="0.0"/>
-  </inertial>
-  <visual>
-    <origin xyz="0.0323 -0.088295 -0.089446" rpy="0 0 0"/>
+    <origin xyz="0.033096700645355887 -0.031000479859321393 0.0028238611176841927" rpy="0 0 0"/>
+    <mass value="0.30666683235154446"/>
+    <inertia ixx="0.000189" iyy="0.000213" izz="0.0004" ixy="-0.0" iyz="-0.0" ixz="-4e-06"/>
+  </inertial>
+  <visual>
+    <origin xyz="-0.089845 -0.03215 -0.089446" rpy="0 0 0"/>
     <geometry>
       <mesh filename="package://robocop_description/meshes/soporteCamara_v2_1.stl" scale="0.001 0.001 0.001"/>
@@ -40,5 +40,5 @@
   </visual>
   <collision>
-    <origin xyz="0.0323 -0.088295 -0.089446" rpy="0 0 0"/>
+    <origin xyz="-0.089845 -0.03215 -0.089446" rpy="0 0 0"/>
     <geometry>
       <mesh filename="package://robocop_description/meshes/soporteCamara_v2_1.stl" scale="0.001 0.001 0.001"/>
@@ -48,10 +48,10 @@
 <link name="depthCamera_v1_1">
   <inertial>
-    <origin xyz="1.2977962637454295e-05 -0.013660026041507928 0.013865360448962805" rpy="0 0 0"/>
-    <mass value="1.4328260381707594"/>
-    <inertia ixx="0.000283" iyy="0.003111" izz="0.00318" ixy="-0.0" iyz="-5e-06" ixz="-0.0"/>
-  </inertial>
-  <visual>
-    <origin xyz="0.0013 -0.16362 -0.097912" rpy="0 0 0"/>
+    <origin xyz="-0.006184113912021172 -1.3611701263174228e-05 0.014463487875515435" rpy="0 0 0"/>
+    <mass value="1.4328263704058224"/>
+    <inertia ixx="0.003111" iyy="0.000283" izz="0.00318" ixy="0.0" iyz="0.0" ixz="-5e-06"/>
+  </inertial>
+  <visual>
+    <origin xyz="-0.157196 -0.00115 -0.097274" rpy="0 0 0"/>
     <geometry>
       <mesh filename="package://robocop_description/meshes/depthCamera_v1_1.stl" scale="0.001 0.001 0.001"/>
@@ -60,5 +60,5 @@
   </visual>
   <collision>
-    <origin xyz="0.0013 -0.16362 -0.097912" rpy="0 0 0"/>
+    <origin xyz="-0.157196 -0.00115 -0.097274" rpy="0 0 0"/>
     <geometry>
       <mesh filename="package://robocop_description/meshes/depthCamera_v1_1.stl" scale="0.001 0.001 0.001"/>
@@ -68,10 +68,10 @@
 <link name="soporteElectronica_v7_1">
   <inertial>
-    <origin xyz="0.07505332529276447 0.055002349444357466 0.04613612305196724" rpy="0 0 0"/>
-    <mass value="1.7280541618979528"/>
-    <inertia ixx="0.002669" iyy="0.008802" izz="0.009606" ixy="0.0" iyz="-0.0" ixz="2.2e-05"/>
-  </inertial>
-  <visual>
-    <origin xyz="0.077 0.056705 -0.089446" rpy="0 0 0"/>
+    <origin xyz="0.0550026777716467 -0.0750539566858314 0.04613612305196782" rpy="0 0 0"/>
+    <mass value="1.7280541618979188"/>
+    <inertia ixx="0.008802" iyy="0.002669" izz="0.009606" ixy="-0.0" iyz="-2.2e-05" ixz="-0.0"/>
+  </inertial>
+  <visual>
+    <origin xyz="0.055155 -0.07685 -0.089446" rpy="0 0 0"/>
     <geometry>
       <mesh filename="package://robocop_description/meshes/soporteElectronica_v7_1.stl" scale="0.001 0.001 0.001"/>
@@ -80,5 +80,5 @@
   </visual>
   <collision>
-    <origin xyz="0.077 0.056705 -0.089446" rpy="0 0 0"/>
+    <origin xyz="0.055155 -0.07685 -0.089446" rpy="0 0 0"/>
     <geometry>
       <mesh filename="package://robocop_description/meshes/soporteElectronica_v7_1.stl" scale="0.001 0.001 0.001"/>
@@ -88,10 +88,10 @@
 <link name="basePrincipal_v4_1">
   <inertial>
-    <origin xyz="0.0674998484671067 -0.09000047986017973 -0.0009996705328835231" rpy="0 0 0"/>
+    <origin xyz="-0.10000015153288912 -4.798601768295652e-07 -0.0009996705328831484" rpy="0 0 0"/>
     <mass value="0.44398234905881495"/>
-    <inertia ixx="0.001466" iyy="0.000868" izz="0.002334" ixy="-0.0" iyz="0.0" ixz="0.0"/>
-  </inertial>
-  <visual>
-    <origin xyz="0.0688 -0.088295 -0.084446" rpy="0 0 0"/>
+    <inertia ixx="0.000868" iyy="0.001466" izz="0.002334" ixy="0.0" iyz="0.0" ixz="0.0"/>
+  </inertial>
+  <visual>
+    <origin xyz="-0.099845 -0.00115 -0.084446" rpy="0 0 0"/>
     <geometry>
       <mesh filename="package://robocop_description/meshes/basePrincipal_v4_1.stl" scale="0.001 0.001 0.001"/>
@@ -100,5 +100,5 @@
   </visual>
   <collision>
-    <origin xyz="0.0688 -0.088295 -0.084446" rpy="0 0 0"/>
+    <origin xyz="-0.099845 -0.00115 -0.084446" rpy="0 0 0"/>
     <geometry>
       <mesh filename="package://robocop_description/meshes/basePrincipal_v4_1.stl" scale="0.001 0.001 0.001"/>
@@ -108,10 +108,10 @@
 <link name="baseRuedas_v3__1__1">
   <inertial>
-    <origin xyz="-0.0029159415133633293 -0.0001620061829542209 -0.035178126681478745" rpy="0 0 0"/>
-    <mass value="0.25465013251117524"/>
-    <inertia ixx="0.001194" iyy="0.000128" izz="0.001072" ixy="-0.0" iyz="4e-06" ixz="-9e-06"/>
-  </inertial>
-  <visual>
-    <origin xyz="0.0763 0.001705 -0.082446" rpy="0 0 0"/>
+    <origin xyz="-0.00016167785566641627 0.002915310120291753 -0.03517812668147839" rpy="0 0 0"/>
+    <mass value="0.25465013251117774"/>
+    <inertia ixx="0.000128" iyy="0.001194" izz="0.001072" ixy="0.0" iyz="9e-06" ixz="4e-06"/>
+  </inertial>
+  <visual>
+    <origin xyz="0.000155 -0.07615 -0.082446" rpy="0 0 0"/>
     <geometry>
       <mesh filename="package://robocop_description/meshes/baseRuedas_v3__1__1.stl" scale="0.001 0.001 0.001"/>
@@ -120,5 +120,5 @@
   </visual>
   <collision>
-    <origin xyz="0.0763 0.001705 -0.082446" rpy="0 0 0"/>
+    <origin xyz="0.000155 -0.07615 -0.082446" rpy="0 0 0"/>
     <geometry>
       <mesh filename="package://robocop_description/meshes/baseRuedas_v3__1__1.stl" scale="0.001 0.001 0.001"/>
@@ -128,10 +128,10 @@
 <link name="baseRuedas_v3_1">
   <inertial>
-    <origin xyz="0.003915638447583289 0.0001610464625932985 -0.035178126681478884" rpy="0 0 0"/>
-    <mass value="0.25465013251117524"/>
-    <inertia ixx="0.001194" iyy="0.000128" izz="0.001072" ixy="-0.0" iyz="-4e-06" ixz="9e-06"/>
-  </inertial>
-  <visual>
-    <origin xyz="-0.0737 0.001705 -0.082446" rpy="0 0 0"/>
+    <origin xyz="0.0001613747898826616 -0.0029162698406539483 -0.03517812668147681" rpy="0 0 0"/>
+    <mass value="0.2546501325111777"/>
+    <inertia ixx="0.000128" iyy="0.001194" izz="0.001072" ixy="0.0" iyz="-9e-06" ixz="-4e-06"/>
+  </inertial>
+  <visual>
+    <origin xyz="0.000155 0.07385 -0.082446" rpy="0 0 0"/>
     <geometry>
       <mesh filename="package://robocop_description/meshes/baseRuedas_v3_1.stl" scale="0.001 0.001 0.001"/>
@@ -140,5 +140,5 @@
   </visual>
   <collision>
-    <origin xyz="-0.0737 0.001705 -0.082446" rpy="0 0 0"/>
+    <origin xyz="0.000155 0.07385 -0.082446" rpy="0 0 0"/>
     <geometry>
       <mesh filename="package://robocop_description/meshes/baseRuedas_v3_1.stl" scale="0.001 0.001 0.001"/>
@@ -148,10 +148,10 @@
 <link name="soportePantalla_v11_1">
   <inertial>
-    <origin xyz="0.0310236963188651 -0.054820451543081225 0.04169322204509168" rpy="0 0 0"/>
-    <mass value="1.4723320792485302"/>
-    <inertia ixx="0.003175" iyy="0.003919" izz="0.002641" ixy="-1e-06" iyz="0.000192" ixz="1e-06"/>
-  </inertial>
-  <visual>
-    <origin xyz="0.0323 0.091705 -0.089446" rpy="0 0 0"/>
+    <origin xyz="-0.05482012321579245 -0.031024327711935747 0.0416932220450911" rpy="0 0 0"/>
+    <mass value="1.4723320792485377"/>
+    <inertia ixx="0.003919" iyy="0.003175" izz="0.002641" ixy="1e-06" iyz="-1e-06" ixz="0.000192"/>
+  </inertial>
+  <visual>
+    <origin xyz="0.090155 -0.03215 -0.089446" rpy="0 0 0"/>
     <geometry>
       <mesh filename="package://robocop_description/meshes/soportePantalla_v11_1.stl" scale="0.001 0.001 0.001"/>
@@ -160,5 +160,5 @@
   </visual>
   <collision>
-    <origin xyz="0.0323 0.091705 -0.089446" rpy="0 0 0"/>
+    <origin xyz="0.090155 -0.03215 -0.089446" rpy="0 0 0"/>
     <geometry>
       <mesh filename="package://robocop_description/meshes/soportePantalla_v11_1.stl" scale="0.001 0.001 0.001"/>
@@ -168,10 +168,10 @@
 <link name="pantallaTouch_v1_1">
   <inertial>
-    <origin xyz="0.057008775248030316 -0.021370109057047254 -0.03552722997181007" rpy="0 0 0"/>
-    <mass value="0.4448049684188369"/>
-    <inertia ixx="0.000218" iyy="0.000719" izz="0.00059" ixy="0.0" iyz="-8.6e-05" ixz="0.0"/>
-  </inertial>
-  <visual>
-    <origin xyz="0.0583 0.13788 -0.223781" rpy="0 0 0"/>
+    <origin xyz="0.014227140264907762 -5.948022128042757e-05 0.03533424485444281" rpy="0 0 0"/>
+    <mass value="0.4448110745769616"/>
+    <inertia ixx="0.000719" iyy="0.000218" izz="0.00059" ixy="-0.0" iyz="-0.0" ixz="-8.6e-05"/>
+  </inertial>
+  <visual>
+    <origin xyz="0.172151 -0.00115 -0.152249" rpy="0 0 0"/>
     <geometry>
       <mesh filename="package://robocop_description/meshes/pantallaTouch_v1_1.stl" scale="0.001 0.001 0.001"/>
@@ -180,5 +180,5 @@
   </visual>
   <collision>
-    <origin xyz="0.0583 0.13788 -0.223781" rpy="0 0 0"/>
+    <origin xyz="0.172151 -0.00115 -0.152249" rpy="0 0 0"/>
     <geometry>
       <mesh filename="package://robocop_description/meshes/pantallaTouch_v1_1.stl" scale="0.001 0.001 0.001"/>
@@ -188,10 +188,10 @@
 <link name="rueda_v2__9__1">
   <inertial>
-    <origin xyz="-0.024841634669981155 -3.770514719891871e-08 9.779884919958182e-08" rpy="0 0 0"/>
-    <mass value="0.03535675163245145"/>
-    <inertia ixx="5e-06" iyy="6e-06" izz="6e-06" ixy="-0.0" iyz="-0.0" ixz="-0.0"/>
-  </inertial>
-  <visual>
-    <origin xyz="0.0793 -0.104667 -0.033913" rpy="0 0 0"/>
+    <origin xyz="2.906220757936673e-07 0.024841003276909218 9.779888714145368e-08" rpy="0 0 0"/>
+    <mass value="0.03535675163245143"/>
+    <inertia ixx="6e-06" iyy="5e-06" izz="6e-06" ixy="0.0" iyz="0.0" ixz="-0.0"/>
+  </inertial>
+  <visual>
+    <origin xyz="-0.106217 -0.07915 -0.033913" rpy="0 0 0"/>
     <geometry>
       <mesh filename="package://robocop_description/meshes/rueda_v2__9__1.stl" scale="0.001 0.001 0.001"/>
@@ -200,5 +200,5 @@
   </visual>
   <collision>
-    <origin xyz="0.0793 -0.104667 -0.033913" rpy="0 0 0"/>
+    <origin xyz="-0.106217 -0.07915 -0.033913" rpy="0 0 0"/>
     <geometry>
       <mesh filename="package://robocop_description/meshes/rueda_v2__9__1.stl" scale="0.001 0.001 0.001"/>
@@ -208,10 +208,10 @@
 <link name="rueda_v2__8__1">
   <inertial>
-    <origin xyz="-0.02484163466998078 -4.79860167851287e-07 3.294670629823415e-07" rpy="0 0 0"/>
-    <mass value="0.03535675163245145"/>
-    <inertia ixx="5e-06" iyy="6e-06" izz="6e-06" ixy="-0.0" iyz="-0.0" ixz="-0.0"/>
-  </inertial>
-  <visual>
-    <origin xyz="0.0793 -0.048295 -0.019446" rpy="0 0 0"/>
+    <origin xyz="-1.5153294408154494e-07 0.024841003276908996 3.2946710029971293e-07" rpy="0 0 0"/>
+    <mass value="0.035356751632451444"/>
+    <inertia ixx="6e-06" iyy="5e-06" izz="6e-06" ixy="0.0" iyz="0.0" ixz="-0.0"/>
+  </inertial>
+  <visual>
+    <origin xyz="-0.049845 -0.07915 -0.019446" rpy="0 0 0"/>
     <geometry>
       <mesh filename="package://robocop_description/meshes/rueda_v2__8__1.stl" scale="0.001 0.001 0.001"/>
@@ -220,5 +220,5 @@
   </visual>
   <collision>
-    <origin xyz="0.0793 -0.048295 -0.019446" rpy="0 0 0"/>
+    <origin xyz="-0.049845 -0.07915 -0.019446" rpy="0 0 0"/>
     <geometry>
       <mesh filename="package://robocop_description/meshes/rueda_v2__8__1.stl" scale="0.001 0.001 0.001"/>
@@ -228,10 +228,10 @@
 <link name="rueda_v2__7__1">
   <inertial>
-    <origin xyz="-0.02484163466997956 -4.798601685970013e-07 3.294670627949914e-07" rpy="0 0 0"/>
-    <mass value="0.03535675163245145"/>
-    <inertia ixx="5e-06" iyy="6e-06" izz="6e-06" ixy="-0.0" iyz="-0.0" ixz="-0.0"/>
-  </inertial>
-  <visual>
-    <origin xyz="0.0793 0.001705 -0.019446" rpy="0 0 0"/>
+    <origin xyz="-1.51532944086722e-07 0.024841003276907747 3.2946710064665763e-07" rpy="0 0 0"/>
+    <mass value="0.03535675163245133"/>
+    <inertia ixx="6e-06" iyy="5e-06" izz="6e-06" ixy="0.0" iyz="0.0" ixz="-0.0"/>
+  </inertial>
+  <visual>
+    <origin xyz="0.000155 -0.07915 -0.019446" rpy="0 0 0"/>
     <geometry>
       <mesh filename="package://robocop_description/meshes/rueda_v2__7__1.stl" scale="0.001 0.001 0.001"/>
@@ -240,5 +240,5 @@
   </visual>
   <collision>
-    <origin xyz="0.0793 0.001705 -0.019446" rpy="0 0 0"/>
+    <origin xyz="0.000155 -0.07915 -0.019446" rpy="0 0 0"/>
     <geometry>
       <mesh filename="package://robocop_description/meshes/rueda_v2__7__1.stl" scale="0.001 0.001 0.001"/>
@@ -248,10 +248,10 @@
 <link name="rueda_v2__6__1">
   <inertial>
-    <origin xyz="-0.02484163466997924 -4.798601688643656e-07 3.29467063017036e-07" rpy="0 0 0"/>
-    <mass value="0.03535675163245145"/>
-    <inertia ixx="5e-06" iyy="6e-06" izz="6e-06" ixy="-0.0" iyz="-0.0" ixz="-0.0"/>
-  </inertial>
-  <visual>
-    <origin xyz="0.0793 0.051705 -0.019446" rpy="0 0 0"/>
+    <origin xyz="-1.5153294388031702e-07 0.024841003276907095 3.294671006501271e-07" rpy="0 0 0"/>
+    <mass value="0.035356751632451625"/>
+    <inertia ixx="6e-06" iyy="5e-06" izz="6e-06" ixy="0.0" iyz="0.0" ixz="-0.0"/>
+  </inertial>
+  <visual>
+    <origin xyz="0.050155 -0.07915 -0.019446" rpy="0 0 0"/>
     <geometry>
       <mesh filename="package://robocop_description/meshes/rueda_v2__6__1.stl" scale="0.001 0.001 0.001"/>
@@ -260,5 +260,5 @@
   </visual>
   <collision>
-    <origin xyz="0.0793 0.051705 -0.019446" rpy="0 0 0"/>
+    <origin xyz="0.050155 -0.07915 -0.019446" rpy="0 0 0"/>
     <geometry>
       <mesh filename="package://robocop_description/meshes/rueda_v2__6__1.stl" scale="0.001 0.001 0.001"/>
@@ -268,10 +268,10 @@
 <link name="rueda_v2__5__1">
   <inertial>
-    <origin xyz="-0.024841634669977394 -4.798601686839543e-07 3.2946706300662765e-07" rpy="0 0 0"/>
-    <mass value="0.03535675163245145"/>
-    <inertia ixx="5e-06" iyy="6e-06" izz="6e-06" ixy="-0.0" iyz="-0.0" ixz="-0.0"/>
-  </inertial>
-  <visual>
-    <origin xyz="0.0793 0.101705 -0.032446" rpy="0 0 0"/>
+    <origin xyz="-1.515329439011337e-07 0.02484100327690518 3.2946710078890495e-07" rpy="0 0 0"/>
+    <mass value="0.035356751632451444"/>
+    <inertia ixx="6e-06" iyy="5e-06" izz="6e-06" ixy="0.0" iyz="0.0" ixz="-0.0"/>
+  </inertial>
+  <visual>
+    <origin xyz="0.100155 -0.07915 -0.032446" rpy="0 0 0"/>
     <geometry>
       <mesh filename="package://robocop_description/meshes/rueda_v2__5__1.stl" scale="0.001 0.001 0.001"/>
@@ -280,5 +280,5 @@
   </visual>
   <collision>
-    <origin xyz="0.0793 0.101705 -0.032446" rpy="0 0 0"/>
+    <origin xyz="0.100155 -0.07915 -0.032446" rpy="0 0 0"/>
     <geometry>
       <mesh filename="package://robocop_description/meshes/rueda_v2__5__1.stl" scale="0.001 0.001 0.001"/>
@@ -288,10 +288,10 @@
 <link name="rueda_v2__4__1">
   <inertial>
-    <origin xyz="0.024841331604199823 7.798481313492367e-08 9.779895947942263e-08" rpy="0 0 0"/>
-    <mass value="0.03535675163245145"/>
-    <inertia ixx="5e-06" iyy="6e-06" izz="6e-06" ixy="0.0" iyz="0.0" ixz="-0.0"/>
-  </inertial>
-  <visual>
-    <origin xyz="-0.0777 0.108078 -0.033913" rpy="0 0 0"/>
+    <origin xyz="4.0631203772345525e-07 -0.024841962997266487 9.7798914786007e-08" rpy="0 0 0"/>
+    <mass value="0.0353567516324516"/>
+    <inertia ixx="6e-06" iyy="5e-06" izz="6e-06" ixy="-0.0" iyz="-0.0" ixz="-0.0"/>
+  </inertial>
+  <visual>
+    <origin xyz="0.106528 0.07685 -0.033913" rpy="0 0 0"/>
     <geometry>
       <mesh filename="package://robocop_description/meshes/rueda_v2__4__1.stl" scale="0.001 0.001 0.001"/>
@@ -300,5 +300,5 @@
   </visual>
   <collision>
-    <origin xyz="-0.0777 0.108078 -0.033913" rpy="0 0 0"/>
+    <origin xyz="0.106528 0.07685 -0.033913" rpy="0 0 0"/>
     <geometry>
       <mesh filename="package://robocop_description/meshes/rueda_v2__4__1.stl" scale="0.001 0.001 0.001"/>
@@ -308,10 +308,10 @@
 <link name="rueda_v2__3__1">
   <inertial>
-    <origin xyz="0.024841331604199518 -4.798601671712754e-07 3.2946717271054027e-07" rpy="0 0 0"/>
-    <mass value="0.03535675163245145"/>
-    <inertia ixx="5e-06" iyy="6e-06" izz="6e-06" ixy="0.0" iyz="0.0" ixz="-0.0"/>
-  </inertial>
-  <visual>
-    <origin xyz="-0.0777 0.051705 -0.019446" rpy="0 0 0"/>
+    <origin xyz="-1.5153294249253824e-07 -0.024841962997268097 3.2946712819406643e-07" rpy="0 0 0"/>
+    <mass value="0.03535675163245149"/>
+    <inertia ixx="6e-06" iyy="5e-06" izz="6e-06" ixy="-0.0" iyz="-0.0" ixz="-0.0"/>
+  </inertial>
+  <visual>
+    <origin xyz="0.050155 0.07685 -0.019446" rpy="0 0 0"/>
     <geometry>
       <mesh filename="package://robocop_description/meshes/rueda_v2__3__1.stl" scale="0.001 0.001 0.001"/>
@@ -320,5 +320,5 @@
   </visual>
   <collision>
-    <origin xyz="-0.0777 0.051705 -0.019446" rpy="0 0 0"/>
+    <origin xyz="0.050155 0.07685 -0.019446" rpy="0 0 0"/>
     <geometry>
       <mesh filename="package://robocop_description/meshes/rueda_v2__3__1.stl" scale="0.001 0.001 0.001"/>
@@ -328,10 +328,10 @@
 <link name="rueda_v2__2__1">
   <inertial>
-    <origin xyz="0.024841331604198866 -4.798601663451134e-07 3.2946717246420953e-07" rpy="0 0 0"/>
-    <mass value="0.03535675163245145"/>
-    <inertia ixx="5e-06" iyy="6e-06" izz="6e-06" ixy="0.0" iyz="0.0" ixz="-0.0"/>
-  </inertial>
-  <visual>
-    <origin xyz="-0.0777 0.001705 -0.019446" rpy="0 0 0"/>
+    <origin xyz="-1.515329426141044e-07 -0.024841962997269235 3.2946712833631375e-07" rpy="0 0 0"/>
+    <mass value="0.03535675163245141"/>
+    <inertia ixx="6e-06" iyy="5e-06" izz="6e-06" ixy="-0.0" iyz="-0.0" ixz="-0.0"/>
+  </inertial>
+  <visual>
+    <origin xyz="0.000155 0.07685 -0.019446" rpy="0 0 0"/>
     <geometry>
       <mesh filename="package://robocop_description/meshes/rueda_v2__2__1.stl" scale="0.001 0.001 0.001"/>
@@ -340,5 +340,5 @@
   </visual>
   <collision>
-    <origin xyz="-0.0777 0.001705 -0.019446" rpy="0 0 0"/>
+    <origin xyz="0.000155 0.07685 -0.019446" rpy="0 0 0"/>
     <geometry>
       <mesh filename="package://robocop_description/meshes/rueda_v2__2__1.stl" scale="0.001 0.001 0.001"/>
@@ -348,10 +348,10 @@
 <link name="rueda_v2__1__1">
   <inertial>
-    <origin xyz="0.02484133160419831 -4.798601659430912e-07 3.2946717221440935e-07" rpy="0 0 0"/>
-    <mass value="0.03535675163245145"/>
-    <inertia ixx="5e-06" iyy="6e-06" izz="6e-06" ixy="0.0" iyz="0.0" ixz="-0.0"/>
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